File: hw/zkeeb_kicad/zkeeb_kicad.kicad_pcb (KiCad board)
At the start: 2 copper layers, 368.5 x 182.5 mm, 139 parts, among them J1 Conn_01x02, SW1 SW_Push, U1 SuperMini nRF52840

Commit message: fix: Updates
Routing:
- net GND: track 10.4 -> 27.7 mm, vias 0 -> 1
- net /R1: track 528.2 -> 542.1 mm, vias 22 -> 26
- net /C3: track 458.3 -> 460.9 mm
Other:
- board size 368.5 x 182.5 mm -> 306.5 x 117.5 mm

Commit message: Fixed switch footprints; TODO mounting screwholes etc.
Parts:
- CH1, CH10, CH11, CH12, CH13, CH14, CH15, CH16, CH17, CH18, CH19, CH2, CH20, CH21, CH22, CH23, CH24, CH25, CH26, CH27, CH28, CH29, CH3, CH30, CH31, CH32, CH33, CH34, CH35, CH36, CH37, CH38, CH39, CH4, CH40, CH41, CH42, CH43, CH44, CH45, CH46, CH47, CH48, CH49, CH5, CH50, CH51, CH52, CH53, CH54, CH55, CH56, CH57, CH58, CH59, CH6, CH60, CH61, CH62, CH63, CH64, CH65, CH66, CH67, CH68, CH7, CH8, CH9: footprint ai03-2725 MX_V2 main Gateron_KS33_Hotswap:Gateron-KS33-Hotswap-1U -> ks33_flipped:Gateron-KS33-Hotswap-1U
Routing:
- net /R1: track 542.1 -> 435.2 mm, vias 26 -> 14
- net /C3: track 460.9 -> 398.7 mm, vias 24 -> 18
- net /C0: track 347.0 -> 383.5 mm, vias 8 -> 22
- net /R5: track 465.4 -> 431.3 mm, vias 14 -> 24
- net /R4: track 472.4 -> 503.9 mm, vias 34 -> 30
- net /R2: track 506.0 -> 480.9 mm, vias 43 -> 22
- net /R3: track 479.4 -> 502.1 mm, vias 25 -> 27
- net /R6: track 444.3 -> 423.7 mm, vias 29 -> 28
- net /C6: track 430.1 -> 414.8 mm, vias 13 -> 17
- net /C8: track 180.6 -> 192.6 mm, vias 3 -> 5
- net /C7: track 400.7 -> 389.1 mm, vias 15 -> 17
- net GND: track 27.7 -> 17.2 mm
- net Net-(D68-A): track 18.6 -> 8.31 mm, vias 0 -> 1
- net Net-(D10-A): track 18.6 -> 8.31 mm, vias 0 -> 1
- net Net-(D6-A): track 18.6 -> 8.31 mm, vias 0 -> 1
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