File: hw/zkeeb_kicad/zkeeb_kicad.kicad_sch (KiCad schematic)
At the start: 139 parts, among them J1 Conn_01x02, SW1 SW_Push, U1 SuperMini nRF52840

Commit message: Fixed switch footprints; TODO mounting screwholes etc.
Parts:
- CH1, CH10, CH11, CH12, CH13, CH14, CH15, CH16, CH17, CH18, CH19, CH2, CH20, CH21, CH22, CH23, CH24, CH25, CH26, CH27, CH28, CH29, CH3, CH30, CH31, CH32, CH33, CH34, CH35, CH36, CH37, CH38, CH39, CH4, CH40, CH41, CH42, CH43, CH44, CH45, CH46, CH47, CH48, CH49, CH5, CH50, CH51, CH52, CH53, CH54, CH55, CH56, CH57, CH58, CH59, CH6, CH60, CH61, CH62, CH63, CH64, CH65, CH66, CH67, CH68, CH7, CH8, CH9: footprint ai03-2725 MX_V2 main Gateron_KS33_Hotswap:Gateron-KS33-Hotswap-1U -> ks33_flipped:Gateron-KS33-Hotswap-1U
